File: hardware/IOIO-OTG.sch (EAGLE design)
At the start: 60 parts, among them Q1 IRLML2244, Q2 2N7002PW, Q3 MOSFET-NCHANNELAO3404A, U1 PIC24FJ256GB206, U2 TPS62133RGTT, U3 MIC5216

Commit message: Seed logo
Parts:
- removed LOGO2: SFE_LOGO_FLAME.1_INCH, SparkFun-Aesthetics:SFE_LOGO_FLAME.1_INCH
- removed LOGO4: SFE_LOGO_NAME_FLAME.1_INCH, SparkFun-Aesthetics:SFE_LOGO_NAME_FLAME.1_INCH
Changed lines of the file:
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@@
 <part name="LOGO1" library="SparkFun-Aesthetics" deviceset="OSHW-LOGO" device="S" value="OSHW-LOGOS"/>
 <part name="FRAME2" library="SparkFun-Aesthetics" deviceset="FRAME-LEDGER" device=""/>
-<part name="LOGO2" library="SparkFun-Aesthetics" deviceset="SFE_LOGO_FLAME" device=".1_INCH"/>
-<part name="LOGO4" library="SparkFun-Aesthetics" deviceset="SFE_LOGO_NAME_FLAME" device=".1_INCH"/>
 <part name="JP21" library="SparkFun-Connectors" deviceset="USB-AB" device="CONN-11794" value="AB MICRO USB"/>
 <part name="JP19" library="SparkFun-Connectors" deviceset="JST_2MM_MALE" device="" value="JST"/>
@@
 <instance part="FRAME2" gate="G$1" x="0" y="0"/>
 <instance part="FRAME2" gate="G$2" x="330.2" y="0"/>
-<instance part="LOGO2" gate="G$1" x="309.88" y="22.86"/>
-<instance part="LOGO4" gate="G$1" x="231.14" y="0"/>
 <instance part="JP21" gate="G$1" x="241.3" y="55.88" rot="MR180"/>
 <instance part="JP19" gate="G$1" x="48.26" y="233.68" smashed="yes" rot="R90">

Commit message: SparkFun Logo
Parts:
- added LOGO2: SFE_LOGO_NAME_FLAME.1_INCH, SparkFun-Aesthetics:SFE_LOGO_NAME_FLAME.1_INCH
- added LOGO3: SFE_LOGO_FLAME.1_INCH, SparkFun-Aesthetics:SFE_LOGO_FLAME.1_INCH
Changed lines of the file:
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@@
 <part name="JP21" library="SparkFun-Connectors" deviceset="USB-AB" device="CONN-11794" value="AB MICRO USB"/>
 <part name="JP19" library="SparkFun-Connectors" deviceset="JST_2MM_MALE" device="" value="JST"/>
+<part name="LOGO2" library="SparkFun-Aesthetics" deviceset="SFE_LOGO_NAME_FLAME" device=".1_INCH"/>
+<part name="LOGO3" library="SparkFun-Aesthetics" deviceset="SFE_LOGO_FLAME" device=".1_INCH"/>
 </parts>
 <sheets>
@@
 <attribute name="NAME" x="49.022" y="241.3" size="1.778" layer="95" font="vector" rot="R180"/>
 </instance>
+<instance part="LOGO2" gate="G$1" x="228.6" y="2.54"/>
+<instance part="LOGO3" gate="G$1" x="309.88" y="25.4"/>
 </instances>
 <busses>
