File: hardware/IOIO-OTG.brd (EAGLE design)
At the start: 68.6 x 30.5 mm, 60 parts, among them Q1 IRLML2244, Q2 2N7002PW, Q3 MOSFET-NCHANNELAO3404A, U1 PIC24FJ256GB206, U2 TPS62133RGTT, U3 V_REG_MIC5216

Commit message: Schematic Cleanup
Parts:
- JP1: value VIN -> (none)
- JP2: value 3.3V -> (none)
- JP4: value 5V -> (none)
- U3: value V_REG_MIC5216 -> MIC5216
Changed lines of the file:
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@@
 <setting verticaltext="up"/>
 </settings>
-<grid distance="0.05" unitdist="inch" unit="inch" style="lines" multiple="2" display="yes" altdistance="0.0001" altunitdist="inch" altunit="inch"/>
+<grid distance="0.05" unitdist="inch" unit="inch" style="lines" multiple="2" display="yes" altdistance="0.005" altunitdist="inch" altunit="inch"/>
 <layers>
 <layer number="1" name="Top" color="4" fill="1" visible="yes" active="yes"/>
@@
 <layer number="27" name="tValues" color="7" fill="1" visible="no" active="yes"/>
 <layer number="28" name="bValues" color="7" fill="1" visible="no" active="yes"/>
-<layer number="29" name="tStop" color="7" fill="3" visible="yes" active="yes"/>
+<layer number="29" name="tStop" color="7" fill="3" visible="no" active="yes"/>
 <layer number="30" name="bStop" color="3" fill="6" visible="no" active="yes"/>
 <layer number="31" name="tCream" color="7" fill="4" visible="no" active="yes"/>
@@
 <layer number="47" name="Measures" color="7" fill="1" visible="no" active="yes"/>
 <layer number="48" name="Document" color="7" fill="1" visible="no" active="yes"/>
-<layer number="49" name="Reference" color="7" fill="1" visible="yes" active="yes"/>
+<layer number="49" name="Reference" color="7" fill="1" visible="no" active="yes"/>
 <layer number="50" name="dxf" color="7" fill="1" visible="no" active="yes"/>
 <layer number="51" name="tDocu" color="6" fill="1" visible="yes" active="yes"/>
@@
 <attribute name="PROD_ID" value="CAP-00810" x="31.9278" y="18.6944" size="1.778" layer="27" rot="R45" display="off"/>
 </element>
-<element name="JP2" library="SparkFun" package="1X03" value="3.3V" x="50.8" y="6.35" smashed="yes" rot="R270">
+<element name="JP2" library="SparkFun" package="1X03" value="" x="50.8" y="6.35" smashed="yes" rot="R270">
 <attribute name="NAME" x="52.6288" y="7.6962" size="1.27" layer="25" ratio="10" rot="R270"/>
 <attribute name="VALUE" x="47.625" y="7.62" size="1.27" layer="27" rot="R270"/>
@@
 <attribute name="VALUE" x="50.165" y="7.62" size="1.27" layer="27" rot="R270"/>
 </element>
-<element name="JP4" library="SparkFun" package="1X03" value="5V" x="55.88" y="6.35" smashed="yes" rot="R270">
+<element name="JP4" library="SparkFun" package="1X03" value="" x="55.88" y="6.35" smashed="yes" rot="R270">
 <attribute name="NAME" x="57.7088" y="7.6962" size="1.27" layer="25" ratio="10" rot="R270"/>
 <attribute name="VALUE" x="52.705" y="7.62" size="1.27" layer="27" rot="R270"/>
@@
 <attribute name="PROD_ID" value="NDUC-11157" x="47.005240625" y="23.2765625" size="1.778" layer="27" rot="R180" display="off"/>
 </element>
-<element name="U3" library="SparkFun-PowerIC" package="MSOP8" value="V_REG_MIC5216" x="42.037" y="22.987" smashed="yes" rot="R180">
+<element name="U3" library="SparkFun-PowerIC" package="MSOP8" value="MIC5216" x="42.037" y="22.987" smashed="yes" rot="R180">
 <attribute name="NAME" x="44.577" y="24.257" size="0.4064" layer="25" rot="R270"/>
 <attribute name="VALUE" x="39.497" y="24.257" size="0.4064" layer="27" rot="R270"/>
@@
 <attribute name="VALUE" x="57.15" y="32.385" size="1.27" layer="27" rot="R180"/>
 </element>
-<element name="JP1" library="SparkFun" package="1X03" value="VIN" x="60.96" y="1.27" smashed="yes" rot="R90">
+<element name="JP1" library="SparkFun" package="1X03" value="" x="60.96" y="1.27" smashed="yes" rot="R90">
 <attribute name="NAME" x="59.1312" y="-0.0762" size="1.27" layer="25" ratio="10" rot="R90"/>
 <attribute name="VALUE" x="64.135" y="0" size="1.27" layer="27" rot="R90"/>
