File: hardware/IOIO-OTG.brd (EAGLE design)
At the start: 68.6 x 30.5 mm, 60 parts, among them Q1 IRLML2244, Q2 2N7002PW, Q3 MOSFET-NCHANNELAO3404A, U1 PIC24FJ256GB206, U2 TPS62133RGTT, U3 MIC5216

Commit message: Seed logo
Parts:
- removed LOGO2: SFE_LOGO_FLAME.1_INCH, SparkFun-Aesthetics:SFE_LOGO_FLAME_.1
- removed LOGO4: SFE_LOGO_NAME_FLAME.1_INCH, SparkFun-Aesthetics:SFE_LOGO_NAME_FLAME_.1
- added U$13: (no value), Logo:LOGO_SILK
- added U$15: (no value), Logo:SMALL_SEEED_LOGO
Other:
- board text added: "www.seeedstudio.com"
Changed lines of the file:
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@@
 <layer number="47" name="Measures" color="7" fill="1" visible="no" active="yes"/>
 <layer number="48" name="Document" color="7" fill="1" visible="no" active="yes"/>
-<layer number="49" name="Reference" color="13" fill="1" visible="yes" active="yes"/>
+<layer number="49" name="Reference" color="13" fill="1" visible="no" active="yes"/>
 <layer number="50" name="dxf" color="7" fill="1" visible="no" active="yes"/>
 <layer number="51" name="tDocu" color="6" fill="1" visible="yes" active="yes"/>
@@
 <dimension x1="66.04" y1="2.54" x2="0" y2="2.54" x3="33.02" y3="35.56" textsize="1.016" layer="47" unit="inch"/>
 <dimension x1="68.58" y1="30.48" x2="0" y2="30.48" x3="34.29" y3="38.1" textsize="1.016" layer="47" unit="inch"/>
+<text x="5.334" y="26.416" size="1.4224" layer="22" ratio="18" rot="SMR270">www.seeedstudio.com</text>
 </plain>
 <attributes>
@@
 <element name="LOGO1" library="SparkFun-Aesthetics" package="OSHW-LOGO-S" value="OSHW-LOGOS" x="66.421" y="15.24" rot="MR270"/>
 <element name="FRAME2" library="SparkFun-Aesthetics" package="CREATIVE_COMMONS" value="FRAME-LEDGER" x="5.08" y="-11.43"/>
-<element name="LOGO2" library="SparkFun-Aesthetics" package="SFE_LOGO_FLAME_.1" value="SFE_LOGO_FLAME.1_INCH" x="15.24" y="14.478" smashed="yes" rot="R90"/>
-<element name="LOGO4" library="SparkFun-Aesthetics" package="SFE_LOGO_NAME_FLAME_.1" value="SFE_LOGO_NAME_FLAME.1_INCH" x="6.096" y="20.32" rot="MR270"/>
 <element name="JP21" library="SparkFun-Connectors" package="USB-AB-MICRO-SMD_V03" value="AB MICRO USB" x="66.548" y="10.16" smashed="yes" rot="R180">
 <attribute name="PROD_ID" value="CONN-11794" x="66.548" y="10.16" size="1.778" layer="27" font="vector" ratio="15" rot="R180" display="off"/>
@@
 <attribute name="VALUE" x="65.554859375" y="20.8407" size="0.4064" layer="27" rot="R270"/>
 </element>
+<element name="U$13" library="Logo" package="LOGO_SILK" value="" x="13.97" y="15.24" rot="R90"/>
+<element name="U$15" library="Logo" package="SMALL_SEEED_LOGO" value="" x="1.905" y="15.875" rot="MR270"/>
 </elements>
 <signals>

Commit message: SparkFun Logo
Parts:
- removed U$13: (no value), Logo:LOGO_SILK
- removed U$15: (no value), Logo:SMALL_SEEED_LOGO
- added LOGO2: SFE_LOGO_NAME_FLAME.1_INCH, SparkFun-Aesthetics:SFE_LOGO_NAME_FLAME_.1
- added LOGO3: SFE_LOGO_FLAME.1_INCH, SparkFun-Aesthetics:SFE_LOGO_FLAME_.1
Other:
- board text removed: "www.seeedstudio.com"
Changed lines of the file:
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@@
 <dimension x1="66.04" y1="2.54" x2="0" y2="2.54" x3="33.02" y3="35.56" textsize="1.016" layer="47" unit="inch"/>
 <dimension x1="68.58" y1="30.48" x2="0" y2="30.48" x3="34.29" y3="38.1" textsize="1.016" layer="47" unit="inch"/>
-<text x="5.334" y="26.416" size="1.4224" layer="22" ratio="18" rot="SMR270">www.seeedstudio.com</text>
 </plain>
 <attributes>
@@
 <attribute name="VALUE" x="65.554859375" y="20.8407" size="0.4064" layer="27" rot="R270"/>
 </element>
-<element name="U$13" library="Logo" package="LOGO_SILK" value="" x="13.97" y="15.24" rot="R90"/>
-<element name="U$15" library="Logo" package="SMALL_SEEED_LOGO" value="" x="1.905" y="15.875" rot="MR270"/>
+<element name="LOGO2" library="SparkFun-Aesthetics" package="SFE_LOGO_NAME_FLAME_.1" value="SFE_LOGO_NAME_FLAME.1_INCH" x="5.715" y="21.59" rot="MR270"/>
+<element name="LOGO3" library="SparkFun-Aesthetics" package="SFE_LOGO_FLAME_.1" value="SFE_LOGO_FLAME.1_INCH" x="14.859" y="14.986" rot="R90"/>
 </elements>
 <signals>
